File: hardware/pcb/luma.kicad_sch (KiCad schematic)
At the start: 89 parts, among them J1 Conn_01x03, Q1 SS8050, Q2 SS8050, SW1 SW_Push, SW2 SW_Push, U1 ESP32-WROOM-32E(8MB), U15 FAN48610BUC50X, U2 USBLC6-2SC6, U6 CP2102N-Axx-xQFN28

Commit message: added stuff
Parts:
- added D13, D14, D15, D16, D17, D18, D19: SK6812, LED_SMD:LED_SK6812_PLCC4_5.0x5.0mm_P3.2mm, symbol LED:SK6812
Connections:
- net +5V: now also D13.3 (VDD), D14.3 (VDD), D15.3 (VDD), D16.3 (VDD), D17.3 (VDD), D18.3 (VDD), D19.3 (VDD)
- net GND: now also D13.1 (VSS), D14.1 (VSS), D15.1 (VSS), D16.1 (VSS), D17.1 (VSS), D18.1 (VSS), D19.1 (VSS)
- net at D12.4 (DOUT): now also D17.2 (DIN)
- new net: D16.2 (DIN), D17.4 (DOUT)
- new net: D13.2 (DIN), D14.4 (DOUT)
- new net: D13.4 (DOUT), D19.2 (DIN)
- new net: D18.2 (DIN), D19.4 (DOUT)
- new net: D14.2 (DIN), D15.4 (DOUT)
- new net: D15.2 (DIN), D16.4 (DOUT)
- no-connect marks 24 -> 23
