File: hardware/pcb/luma.kicad_sch (KiCad schematic)
At the start: 81 parts, among them J1 Conn_01x03, J2 Conn_01x03_Pin, Q1 SS8050, Q2 SS8050, SW1 SW_Push, SW2 SW_Push, U1 ESP32-WROOM-32E(8MB), U15 FAN48610BUC50X, U2 USBLC6-2SC6, U6 CP2102N-Axx-xQFN28

Commit message: prod
Parts:
- SW1, SW2: LCSC (none) -> C720477
Changed lines of the file:
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@@
+			)
+		)
+		(property "LCSC" "C720477"
+			(at 302.26 52.07 0)
+			(effects
+				(font
+					(size 1.27 1.27)
+				)
+				(hide yes)
 			)
 		)
@@
 			(at 302.26 36.83 0)
 			(effects
+				(font
+					(size 1.27 1.27)
+				)
+				(hide yes)
+			)
+		)
+		(property "LCSC" "C720477"
+			(at 302.26 36.83 0)
+			(effects
