File: hardware/pcb/luma.kicad_pcb (KiCad board)
At the start: 2 copper layers, 58 x 58 mm, 89 parts, among them J1 Conn_01x03, Q1 SS8050, Q2 SS8050, SW1 SW_Push, SW2 SW_Push, U1 ESP32-WROOM-32E(8MB), U15 FAN48610BUC50X, U2 USBLC6-2SC6, U6 CP2102N-Axx-xQFN28

Commit message: added stuff
Parts:
- added D13: SK6812, LED_SMD:LED_SK6812_PLCC4_5.0x5.0mm_P3.2mm, B.Cu at (153.2, 123.2)
- added D14: SK6812, LED_SMD:LED_SK6812_PLCC4_5.0x5.0mm_P3.2mm, B.Cu at (153.2, 116.6)
- added D15: SK6812, LED_SMD:LED_SK6812_PLCC4_5.0x5.0mm_P3.2mm, B.Cu at (153.2, 110.0)
- added D16: SK6812, LED_SMD:LED_SK6812_PLCC4_5.0x5.0mm_P3.2mm, B.Cu at (153.2, 103.4)
- added D17: SK6812, LED_SMD:LED_SK6812_PLCC4_5.0x5.0mm_P3.2mm, B.Cu at (153.2, 96.7)
- added D18: SK6812, LED_SMD:LED_SK6812_PLCC4_5.0x5.0mm_P3.2mm, B.Cu at (153.2, 90.1)
- added D19: SK6812, LED_SMD:LED_SK6812_PLCC4_5.0x5.0mm_P3.2mm, B.Cu at (153.2, 83.5)
Connections:
- D12 pad 4: unconnected-(D12-DOUT-Pad4) -> Net-(D12-DOUT)
Routing:
- net /BOOT: track 0.00 -> 63.4 mm
- net VBUS: track 33.9 -> 87.3 mm, vias 5 -> 9
- net /I2C_SCL: track 1.63 -> 52.5 mm, vias 0 -> 3
- net /I2C_SDA: track 1.62 -> 52.0 mm, vias 0 -> 5
- net /RXD: track 0.00 -> 42.4 mm, vias 0 -> 2
- net /TXD: track 0.00 -> 41.4 mm, vias 0 -> 2
- net +3.3V: track 104.4 -> 143.7 mm, vias 3 -> 5
- net +5V: track 206.7 -> 241.7 mm
- net Net-(J1-Pin_2): track 44.8 -> 64.6 mm
- net /EN: track 0.00 -> 19.0 mm, vias 0 -> 2
- net GND: track 85.1 -> 103.4 mm, vias 12 -> 49
- net +BATT: track 51.4 -> 69.0 mm
- net /LED: track 0.00 -> 17.1 mm, vias 0 -> 1
- net Net-(U3-REGN): track 15.7 -> 20.5 mm
- net Net-(Q1-B): track 5.10 -> 7.03 mm, vias 0 -> 2
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- added copper zone on F.Cu, net GND

Commit message: finished!
Parts:
- removed D10, D11, D12, D13, D14, D15, D16, D17, D18, D19, D4, D5, D6, D7, D8, D9: SK6812, LED_SMD:LED_SK6812_PLCC4_5.0x5.0mm_P3.2mm
- added J2: Conn_01x03_Pin, Connector_PinHeader_2.00mm:PinHeader_1x03_P2.00mm_Vertical, F.Cu at (187.4, 103.2)
- R42: value 10m -> WW25WR010FTL; footprint Resistor_SMD:R_0402_1005Metric -> luma:R2512
- moved R9 44.3 mm to (186.9, 96.6), turned to 90 degrees
- moved SW2 40.9 mm to (189.3, 93.8), turned to -90 degrees
- moved C5 36.4 mm to (191.7, 94.0), turned to -90 degrees
- moved R23 33.6 mm to (216.7, 112.5), turned to 180 degrees
- moved R21 33.2 mm to (214.6, 112.5), turned to 0 degrees
- moved R5 31.6 mm to (221.8, 109.4), turned to 90 degrees
- moved C4 30.9 mm to (211.1, 111.0), turned to -90 degrees
- moved C3 30.1 mm to (212.4, 110.4), turned to -90 degrees
- moved D3 30.0 mm to (220.3, 108.8), turned to 0 degrees
- moved R4 29.1 mm to (221.8, 107.4), turned to -90 degrees
- moved D2 28.9 mm to (220.3, 107.9), turned to 0 degrees
- moved U6 28.1 mm to (216.1, 108.6), turned to 0 degrees
- moved TP2 25.7 mm to (216.2, 129.1)
- moved TP1 25.7 mm to (219.7, 129.1)
- moved TP3 25.7 mm to (212.6, 129.1)
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Connections:
- R42 pad 1: +BATT -> Net-(U4-SRN)
- R42 pad 2: Net-(U4-SRN) -> +BATT
- U2 pad 1: /DN -> /DP
- U2 pad 3: /DP -> /DN
- U2 pad 4: /D+ -> /D-
- U2 pad 6: /D- -> /D+
Routing:
- net +5V: track 241.7 -> 23.0 mm, vias 1 -> 0
- net GND: track 103.4 -> 55.8 mm, vias 49 -> 45
- net VBUS: track 87.3 -> 54.0 mm, vias 9 -> 4
- net /BOOT: track 63.4 -> 31.5 mm, vias 0 -> 2
- net /EN: track 19.0 -> 47.4 mm
- net +3.3V: track 143.7 -> 117.8 mm, vias 5 -> 11
- net Net-(D10-DIN): track 25.8 -> 0.00 mm
- net Net-(D5-DOUT): track 25.7 -> 0.00 mm
- net Net-(D10-DOUT): track 25.3 -> 0.00 mm
- net /D+: track 44.5 -> 19.5 mm, vias 2 -> 0
- net /D-: track 43.4 -> 18.6 mm, vias 2 -> 0
- net Net-(D11-DOUT): track 23.8 -> 0.00 mm
- net Net-(D6-DOUT): track 23.8 -> 0.00 mm
- net Net-(D12-DIN): track 21.4 -> 0.00 mm, vias 2 -> 0
- net Net-(D8-DOUT): track 21.4 -> 0.00 mm
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Other:
- board size 58 x 58 mm -> 40 x 58 mm
- board text added: "GND 5V LED"
- board text added: "GND TM BAT"

Commit message: fix pcb  placement
Parts:
- moved C6 1.36 mm to (187.0, 86.6)
Routing:
- net /EN: track 47.4 -> 48.6 mm
Changed lines of the file:
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@@
 	(footprint "Capacitor_SMD:C_0402_1005Metric"
 		(layer "F.Cu")
-		(at 187.76 85.45 90)
+		(at 187 86.575 90)
 		(descr "Capacitor SMD 0402 (1005 Metric), square (rectangular) end terminal, IPC-7351 nominal, (Body size source: IPC-SM-782 page 76, https://www.pcb-3d.com/wordpress/wp-content/uploads/ipc-sm-782a_amendment_1_and_2.pdf), generated with kicad-footprint-generator")
 		(tags "capacitor")
@@
 	)
 	(segment
-		(start 195.95 83.7)
-		(end 195.94 83.69)
-		(width 0.6)
+		(start 188.125 84.97)
+		(end 189.36 84.97)
+		(width 0.3)
 		(layer "F.Cu")
 		(net 3)
 	)
 	(segment
-		(start 187.76 84.97)
-		(end 189.36 84.97)
+		(start 189.36 84.97)
+		(end 189.38 84.95)
 		(width 0.3)
 		(layer "F.Cu")
@@
 	)
 	(segment
+		(start 195.95 83.7)
+		(end 195.94 83.69)
+		(width 0.6)
+		(layer "F.Cu")
+		(net 3)
+	)
+	(segment
 		(start 219.53 101.3)
 		(end 219.53 99.87)
@@
 	)
 	(segment
-		(start 189.36 84.97)
-		(end 189.38 84.95)
+		(start 187 86.095)
+		(end 188.125 84.97)
 		(width 0.3)
 		(layer "F.Cu")

Commit message: added tolerances an finished build
Parts:
- moved R2 0.25 mm to (201.2, 121.5)
- moved R1 0.17 mm to (204.9, 121.5)
Changed lines of the file:
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@@
 	(footprint "PCM_Resistor_SMD_AKL:R_0402_1005Metric"
 		(layer "F.Cu")
-		(at 204.73 121.49 90)
+		(at 204.9 121.525 90)
 		(descr "Resistor SMD 0402 (1005 Metric), square (rectangular) end terminal, IPC_7351 nominal, (Body size source: IPC-SM-782 page 72, https://www.pcb-3d.com/wordpress/wp-content/uploads/ipc-sm-782a_amendment_1_and_2.pdf), Alternate KiCad Library")
 		(tags "resistor")
@@
 	(footprint "PCM_Resistor_SMD_AKL:R_0402_1005Metric"
 		(layer "F.Cu")
-		(at 201.4 121.49 90)
+		(at 201.15 121.475 90)
 		(descr "Resistor SMD 0402 (1005 Metric), square (rectangular) end terminal, IPC_7351 nominal, (Body size source: IPC-SM-782 page 72, https://www.pcb-3d.com/wordpress/wp-content/uploads/ipc-sm-782a_amendment_1_and_2.pdf), Alternate KiCad Library")
 		(tags "resistor")
@@
 	)
 	(segment
-		(start 204.85 124.08)
-		(end 204.974 123.956)
+		(start 204.9 124.03)
+		(end 204.9 122.035)
 		(width 0.2)
 		(layer "F.Cu")
@@
 	)
 	(segment
-		(start 204.974 123.956)
-		(end 204.974 122.244)
-		(width 0.2)
-		(layer "F.Cu")
-		(net 35)
-	)
-	(segment
-		(start 204.974 122.244)
-		(end 204.73 122)
+		(start 204.85 124.08)
+		(end 204.9 124.03)
 		(width 0.2)
 		(layer "F.Cu")
@@
 	)
 	(segment
-		(start 201.85 122.45)
-		(end 201.4 122)
+		(start 201.85 122.685)
+		(end 201.15 121.985)
 		(width 0.2)
 		(layer "F.Cu")
@@
 	(segment
 		(start 201.85 124.08)
-		(end 201.85 122.45)
+		(end 201.85 122.685)
 		(width 0.2)
 		(layer "F.Cu")
