File: hardware/pcb/luma-backups/luma_9.kicad_sch (KiCad schematic)
At the start: 81 parts, among them J1 Conn_01x03, J2 Conn_01x03_Pin, Q1 SS8050, Q2 SS8050, SW1 SW_Push, SW2 SW_Push, U1 ESP32-WROOM-32E(8MB), U15 FAN48610BUC50X, U2 USBLC6-2SC6, U6 CP2102N-Axx-xQFN28

Commit message: finished!
Parts:
- removed J2: Conn_01x03_Pin, Connector_PinHeader_2.00mm:PinHeader_1x03_P2.00mm_Vertical, symbol Connector:Conn_01x03_Pin
- removed R42: WW25WR010FTL, luma:R2512, symbol luma:WW25WR010FTL
- added D10, D11, D12, D4, D5, D6, D7, D8, D9: SK6812, LED_SMD:LED_SK6812_PLCC4_5.0x5.0mm_P3.2mm, symbol LED:SK6812
- added R42: 10m, Resistor_SMD:R_0402_1005Metric, symbol Device:R
- U6: LCSC C964632 -> (none)
Connections:
- net +5V: now also D10.3 (VDD), D11.3 (VDD), D12.3 (VDD), D4.3 (VDD), D5.3 (VDD), D6.3 (VDD), D7.3 (VDD), D8.3 (VDD), D9.3 (VDD)
- net +BATT: now also R42.1
- net D+: now also U2.4 (I/O2); no longer U2.6 (I/O1)
- net D-: now also U2.6 (I/O1); no longer U2.4 (I/O2)
- net DN: now also U2.1 (I/O1); no longer U2.3 (I/O2)
- net DP: now also U2.3 (I/O2); no longer U2.1 (I/O1)
- net GND: now also D10.1 (VSS), D11.1 (VSS), D12.1 (VSS), D4.1 (VSS), D5.1 (VSS), D6.1 (VSS), D7.1 (VSS), D8.1 (VSS), D9.1 (VSS)
- net LED: now also D8.2 (DIN)
- net at C61.1, C62.1, U3.13 (BAT)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: now also R42.2
- new net: D8.4 (DOUT), D9.2 (DIN)
- new net: D10.2 (DIN), D9.4 (DOUT)
- new net: D11.4 (DOUT), D4.2 (DIN)
- new net: D4.4 (DOUT), D5.2 (DIN)
- new net: D12.2 (DIN), D7.4 (DOUT)
- new net: D5.4 (DOUT), D6.2 (DIN)
- new net: D6.4 (DOUT), D7.2 (DIN)
- new net: D10.4 (DOUT), D11.2 (DIN)
- no-connect marks 43 -> 24
